Commit message: feat: add gripper trajectory execution support

File: my_robot_description/urdf/common_properties.xacro (robot description, xacro)
@@ -7,3 +7,9 @@
         <color rgba="0.0 0.0 0.5 1.0" />
     </material>
+    <material name="dark_green">
+        <color rgba="0.0 0.4 0.0 1.0" />
+    </material>
+    <material name="light_green">
+        <color rgba="0.0 0.6 0.1 1.0" />
+    </material>
 </robot>

File: my_robot_description/urdf/my_robot.urdf.xacro (robot description, xacro)
@@ -3,3 +3,9 @@
     <xacro:include filename="common_properties.xacro" />
     <xacro:include filename="arm.xacro" />
+    <xacro:include filename="gripper.xacro" />
+    <joint name="gripper_base_link" type="fixed">
+        <parent link="tool_link" />
+        <child link="gripper_base_link" />
+        <origin xyz="0.0 0.0 0.0" rpy="0.0 0.0 0.0" />
+    </joint>
 </robot>
